File: KiCad/DAC.sch (KiCad schematic (older format))
At the start: 16 parts

Commit message: PCB v0.2.
Parts:
- R41, R42, R43, R44, R45, R46, R47, R48, R49: value 20K -> 20K 0.1%
- R50, R51, R52, R53, R54, R55, R56: value 10K -> 10K 0.1%
Changed lines of the file:
@@
 P 3300 1900
 F 0 "R50" H 3241 1946 50  0000 R CNN
-F 1 "10K" H 3241 1855 50  0000 R CNN
+F 1 "10K 0.1%" H 3241 1855 50  0000 R CNN
 F 2 "Resistor_SMD:R_0603_1608Metric" H 3300 1900 50  0001 C CNN
 F 3 "~" H 3300 1900 50  0001 C CNN
@@
 P 3050 1300
 F 0 "R41" V 2854 1300 50  0000 C CNN
-F 1 "20K" V 2945 1300 50  0000 C CNN
+F 1 "20K 0.1%" V 2945 1300 50  0000 C CNN
 F 2 "Resistor_SMD:R_0603_1608Metric" H 3050 1300 50  0001 C CNN
 F 3 "~" H 3050 1300 50  0001 C CNN
@@
 P 3050 1650
 F 0 "R42" V 2854 1650 50  0000 C CNN
-F 1 "20K" V 2945 1650 50  0000 C CNN
+F 1 "20K 0.1%" V 2945 1650 50  0000 C CNN
 F 2 "Resistor_SMD:R_0603_1608Metric" H 3050 1650 50  0001 C CNN
 F 3 "~" H 3050 1650 50  0001 C CNN
@@
 P 3300 2300
 F 0 "R51" H 3241 2254 50  0000 R CNN
-F 1 "10K" H 3241 2345 50  0000 R CNN
+F 1 "10K 0.1%" H 3241 2345 50  0000 R CNN
 F 2 "Resistor_SMD:R_0603_1608Metric" H 3300 2300 50  0001 C CNN
 F 3 "~" H 3300 2300 50  0001 C CNN
@@
 P 3050 2050
 F 0 "R43" V 2854 2050 50  0000 C CNN
-F 1 "20K" V 2945 2050 50  0000 C CNN
+F 1 "20K 0.1%" V 2945 2050 50  0000 C CNN
 F 2 "Resistor_SMD:R_0603_1608Metric" H 3050 2050 50  0001 C CNN
 F 3 "~" H 3050 2050 50  0001 C CNN
@@
 P 3300 2700
 F 0 "R52" H 3241 2654 50  0000 R CNN
-F 1 "10K" H 3241 2745 50  0000 R CNN
+F 1 "10K 0.1%" H 3241 2745 50  0000 R CNN
 F 2 "Resistor_SMD:R_0603_1608Metric" H 3300 2700 50  0001 C CNN
 F 3 "~" H 3300 2700 50  0001 C CNN
@@
 P 3050 2450
 F 0 "R44" V 2854 2450 50  0000 C CNN
-F 1 "20K" V 2945 2450 50  0000 C CNN
+F 1 "20K 0.1%" V 2945 2450 50  0000 C CNN
 F 2 "Resistor_SMD:R_0603_1608Metric" H 3050 2450 50  0001 C CNN
 F 3 "~" H 3050 2450 50  0001 C CNN
@@
 P 3300 3100
 F 0 "R53" H 3241 3054 50  0000 R CNN
-F 1 "10K" H 3241 3145 50  0000 R CNN
+F 1 "10K 0.1%" H 3241 3145 50  0000 R CNN
 F 2 "Resistor_SMD:R_0603_1608Metric" H 3300 3100 50  0001 C CNN
 F 3 "~" H 3300 3100 50  0001 C CNN
@@
 P 3050 2850
 F 0 "R45" V 2854 2850 50  0000 C CNN
-F 1 "20K" V 2945 2850 50  0000 C CNN
+F 1 "20K 0.1%" V 2945 2850 50  0000 C CNN
 F 2 "Resistor_SMD:R_0603_1608Metric" H 3050 2850 50  0001 C CNN
 F 3 "~" H 3050 2850 50  0001 C CNN
@@
 P 3300 3500
 F 0 "R54" H 3241 3454 50  0000 R CNN
-F 1 "10K" H 3241 3545 50  0000 R CNN
+F 1 "10K 0.1%" H 3241 3545 50  0000 R CNN
 F 2 "Resistor_SMD:R_0603_1608Metric" H 3300 3500 50  0001 C CNN
 F 3 "~" H 3300 3500 50  0001 C CNN
@@
 P 3050 3250
 F 0 "R46" V 2854 3250 50  0000 C CNN
-F 1 "20K" V 2945 3250 50  0000 C CNN
+F 1 "20K 0.1%" V 2945 3250 50  0000 C CNN
 F 2 "Resistor_SMD:R_0603_1608Metric" H 3050 3250 50  0001 C CNN
 F 3 "~" H 3050 3250 50  0001 C CNN
@@
 P 3300 3900
 F 0 "R55" H 3241 3854 50  0000 R CNN
-F 1 "10K" H 3241 3945 50  0000 R CNN
+F 1 "10K 0.1%" H 3241 3945 50  0000 R CNN
 F 2 "Resistor_SMD:R_0603_1608Metric" H 3300 3900 50  0001 C CNN
 F 3 "~" H 3300 3900 50  0001 C CNN
@@
 P 3050 3650
 F 0 "R47" V 2854 3650 50  0000 C CNN
-F 1 "20K" V 2945 3650 50  0000 C CNN
+F 1 "20K 0.1%" V 2945 3650 50  0000 C CNN
 F 2 "Resistor_SMD:R_0603_1608Metric" H 3050 3650 50  0001 C CNN
 F 3 "~" H 3050 3650 50  0001 C CNN
@@
 P 3300 4300
 F 0 "R56" H 3241 4254 50  0000 R CNN
-F 1 "10K" H 3241 4345 50  0000 R CNN
+F 1 "10K 0.1%" H 3241 4345 50  0000 R CNN
 F 2 "Resistor_SMD:R_0603_1608Metric" H 3300 4300 50  0001 C CNN
 F 3 "~" H 3300 4300 50  0001 C CNN
@@
 P 3050 4050
 F 0 "R48" V 2854 4050 50  0000 C CNN
-F 1 "20K" V 2945 4050 50  0000 C CNN
+F 1 "20K 0.1%" V 2945 4050 50  0000 C CNN
 F 2 "Resistor_SMD:R_0603_1608Metric" H 3050 4050 50  0001 C CNN
 F 3 "~" H 3050 4050 50  0001 C CNN
@@
 P 3050 4450
 F 0 "R49" V 2854 4450 50  0000 C CNN
-F 1 "20K" V 2945 4450 50  0000 C CNN
+F 1 "20K 0.1%" V 2945 4450 50  0000 C CNN
 F 2 "Resistor_SMD:R_0603_1608Metric" H 3050 4450 50  0001 C CNN
 F 3 "~" H 3050 4450 50  0001 C CNN
@@
 P 2800 1350
 F 0 "#PWR0205" H 2800 1100 50  0001 C CNN
-F 1 "GND" H 2805 1177 50  0000 C CNN
+F 1 "GND" H 2750 1200 50  0000 C CNN
 F 2 "" H 2800 1350 50  0001 C CNN
 F 3 "" H 2800 1350 50  0001 C CNN
