File: KiCad/Output.sch (KiCad schematic (older format))
At the start: 21 parts, among them J3 Conn_01x08, U25 74LVC1G04, U26 74LS377

Commit message: PCB v0.2.
Parts:
- D28, D29, D30, D31, D32, D33, D34, D35: value LED_Small -> LED
- J3: value Conn_01x08 -> Out
- U25: value 74LVC1G04 -> SN74LVC1G04DCK
- U26: value 74LS377 -> SN74HC377DW
Changed lines of the file:
@@
 AR Path="/5E38B78E/5E45EB2A" Ref="D28"  Part="1"
 F 0 "D28" H 7500 2700 50  0000 C CNN
-F 1 "LED_Small" H 7150 2700 50  0000 C CNN
+F 1 "LED" H 7150 2700 50  0000 C CNN
 F 2 "LED_SMD:LED_0603_1608Metric" V 7400 2750 50  0001 C CNN
 F 3 "~" V 7400 2750 50  0001 C CNN
@@
 AR Path="/5E38B78E/5E462343" Ref="D35"  Part="1"
 F 0 "D35" H 7500 3400 50  0000 C CNN
-F 1 "LED_Small" H 7150 3400 50  0000 C CNN
+F 1 "LED" H 7150 3400 50  0000 C CNN
 F 2 "LED_SMD:LED_0603_1608Metric" V 7400 3450 50  0001 C CNN
 F 3 "~" V 7400 3450 50  0001 C CNN
@@
 AR Path="/5E38B78E/5E462336" Ref="D34"  Part="1"
 F 0 "D34" H 7500 3300 50  0000 C CNN
-F 1 "LED_Small" H 7150 3300 50  0000 C CNN
+F 1 "LED" H 7150 3300 50  0000 C CNN
 F 2 "LED_SMD:LED_0603_1608Metric" V 7400 3350 50  0001 C CNN
 F 3 "~" V 7400 3350 50  0001 C CNN
@@
 AR Path="/5E38B78E/5E461419" Ref="D33"  Part="1"
 F 0 "D33" H 7500 3200 50  0000 C CNN
-F 1 "LED_Small" H 7150 3200 50  0000 C CNN
+F 1 "LED" H 7150 3200 50  0000 C CNN
 F 2 "LED_SMD:LED_0603_1608Metric" V 7400 3250 50  0001 C CNN
 F 3 "~" V 7400 3250 50  0001 C CNN
@@
 AR Path="/5E38B78E/5E46140C" Ref="D32"  Part="1"
 F 0 "D32" H 7500 3100 50  0000 C CNN
-F 1 "LED_Small" H 7150 3100 50  0000 C CNN
+F 1 "LED" H 7150 3100 50  0000 C CNN
 F 2 "LED_SMD:LED_0603_1608Metric" V 7400 3150 50  0001 C CNN
 F 3 "~" V 7400 3150 50  0001 C CNN
@@
 AR Path="/5E38B78E/5E4601C1" Ref="D31"  Part="1"
 F 0 "D31" H 7500 3000 50  0000 C CNN
-F 1 "LED_Small" H 7150 3000 50  0000 C CNN
+F 1 "LED" H 7150 3000 50  0000 C CNN
 F 2 "LED_SMD:LED_0603_1608Metric" V 7400 3050 50  0001 C CNN
 F 3 "~" V 7400 3050 50  0001 C CNN
@@
 AR Path="/5E38B78E/5E4601B4" Ref="D30"  Part="1"
 F 0 "D30" H 7500 2900 50  0000 C CNN
-F 1 "LED_Small" H 7150 2900 50  0000 C CNN
+F 1 "LED" H 7150 2900 50  0000 C CNN
 F 2 "LED_SMD:LED_0603_1608Metric" V 7400 2950 50  0001 C CNN
 F 3 "~" V 7400 2950 50  0001 C CNN
@@
 AR Path="/5E38B78E/5E45EB37" Ref="D29"  Part="1"
 F 0 "D29" H 7500 2800 50  0000 C CNN
-F 1 "LED_Small" H 7150 2800 50  0000 C CNN
+F 1 "LED" H 7150 2800 50  0000 C CNN
 F 2 "LED_SMD:LED_0603_1608Metric" V 7400 2850 50  0001 C CNN
 F 3 "~" V 7400 2850 50  0001 C CNN
@@
 P 6950 4000
 F 0 "J3" H 7030 3992 50  0000 L CNN
-F 1 "Conn_01x08" H 7030 3901 50  0000 L CNN
+F 1 "Out" H 7030 3901 50  0000 L CNN
 F 2 "Connector_PinHeader_2.54mm:PinHeader_1x08_P2.54mm_Vertical" H 6950 4000 50  0001 C CNN
 F 3 "~" H 6950 4000 50  0001 C CNN
@@
 AR Path="/5E38B78E/60670EC9" Ref="U26"  Part="1"
 F 0 "U26" H 5300 4000 50  0000 C CNN
-F 1 "74LS377" H 5400 3900 50  0000 C CNN
+F 1 "SN74HC377DW" H 5550 3900 50  0000 C CNN
 F 2 "Package_SO:SOIC-20W_7.5x12.8mm_P1.27mm" H 5200 3250 50  0001 C CNN
 F 3 "http://www.ti.com/lit/gpn/sn74LS377" H 5200 3250 50  0001 C CNN
@@
 AR Path="/5E38B78E/606A0A0B" Ref="U25"  Part="1"
 F 0 "U25" H 4500 4950 50  0000 C CNN
-F 1 "74LVC1G04" H 4650 4650 50  0000 C CNN
+F 1 "SN74LVC1G04DCK" H 4750 4650 50  0000 C CNN
 F 2 "Package_TO_SOT_SMD:SOT-353_SC-70-5" H 4350 4750 50  0001 C CNN
 F 3 "http://www.ti.com/lit/sg/scyt129e/scyt129e.pdf" H 4350 4750 50  0001 C CNN

Commit message: v0.3 Changed to Schmitt-Trigger ICs Added pull-down resistor to Clock Enable
Parts:
- R28, R29, R30, R31, R32, R33, R34, R35: value rled -> 39K
Changed lines of the file:
@@
 Sheet 4 9
 Title "Schilk_SA-ADC"
-Date "2020-02-03"
-Rev "v0.0 (Prod.)"
+Date "2020-08-26"
+Rev "v0.3"
 Comp ""
 Comment1 ""
@@
 AR Path="/5E38B78E/5E45EB24" Ref="R28"  Part="1"
 F 0 "R28" V 6900 2950 50  0000 C CNN
-F 1 "rled" V 6900 2550 50  0000 C CNN
+F 1 "39K" V 6900 2550 50  0000 C CNN
 F 2 "Resistor_SMD:R_0603_1608Metric" H 6950 2750 50  0001 C CNN
 F 3 "~" H 6950 2750 50  0001 C CNN
@@
 AR Path="/5E38B78E/5E45EB31" Ref="R29"  Part="1"
 F 0 "R29" V 6900 3050 50  0000 C CNN
-F 1 "rled" V 6900 2650 50  0000 C CNN
+F 1 "39K" V 6900 2650 50  0000 C CNN
 F 2 "Resistor_SMD:R_0603_1608Metric" H 6950 2850 50  0001 C CNN
 F 3 "~" H 6950 2850 50  0001 C CNN
@@
 AR Path="/5E38B78E/5E4601AE" Ref="R30"  Part="1"
 F 0 "R30" V 6900 3150 50  0000 C CNN
-F 1 "rled" V 6900 2750 50  0000 C CNN
+F 1 "39K" V 6900 2750 50  0000 C CNN
 F 2 "Resistor_SMD:R_0603_1608Metric" H 6950 2950 50  0001 C CNN
 F 3 "~" H 6950 2950 50  0001 C CNN
@@
 AR Path="/5E38B78E/5E4601BB" Ref="R31"  Part="1"
 F 0 "R31" V 6900 3250 50  0000 C CNN
-F 1 "rled" V 6900 2850 50  0000 C CNN
+F 1 "39K" V 6900 2850 50  0000 C CNN
 F 2 "Resistor_SMD:R_0603_1608Metric" H 6950 3050 50  0001 C CNN
 F 3 "~" H 6950 3050 50  0001 C CNN
@@
 AR Path="/5E38B78E/5E461406" Ref="R32"  Part="1"
 F 0 "R32" V 6900 3350 50  0000 C CNN
-F 1 "rled" V 6900 2950 50  0000 C CNN
+F 1 "39K" V 6900 2950 50  0000 C CNN
 F 2 "Resistor_SMD:R_0603_1608Metric" H 6950 3150 50  0001 C CNN
 F 3 "~" H 6950 3150 50  0001 C CNN
@@
 AR Path="/5E38B78E/5E461413" Ref="R33"  Part="1"
 F 0 "R33" V 6900 3450 50  0000 C CNN
-F 1 "rled" V 6900 3050 50  0000 C CNN
+F 1 "39K" V 6900 3050 50  0000 C CNN
 F 2 "Resistor_SMD:R_0603_1608Metric" H 6950 3250 50  0001 C CNN
 F 3 "~" H 6950 3250 50  0001 C CNN
@@
 AR Path="/5E38B78E/5E462330" Ref="R34"  Part="1"
 F 0 "R34" V 6900 3550 50  0000 C CNN
-F 1 "rled" V 6900 3150 50  0000 C CNN
+F 1 "39K" V 6900 3150 50  0000 C CNN
 F 2 "Resistor_SMD:R_0603_1608Metric" H 6950 3350 50  0001 C CNN
 F 3 "~" H 6950 3350 50  0001 C CNN
@@
 AR Path="/5E38B78E/5E46233D" Ref="R35"  Part="1"
 F 0 "R35" V 6900 3650 50  0000 C CNN
-F 1 "rled" V 6900 3250 50  0000 C CNN
+F 1 "39K" V 6900 3250 50  0000 C CNN
 F 2 "Resistor_SMD:R_0603_1608Metric" H 6950 3450 50  0001 C CNN
 F 3 "~" H 6950 3450 50  0001 C CNN
