File: KiCad/PWR.sch (KiCad schematic (older format))
At the start: 9 parts, among them J2 Conn_01x02, U37 LM317L_TO92, U38 L7805

Commit message: fixed small typos
Other:
- note added: "OpAmp used as comparator\nneeds supply slightly higher than 5v to compare signals close to / at 5v.\n\nSpecific voltage was choosen as it both enabled comparing accross\nthe whole 0-5v band, and resulted in the opamp outputing around 5V as\nlogic-high. (Output of Opamp ist at max aprox. 1.2-1.3 V lower than Supply Voltage)"
- note removed: "OpAmp used as comparator\n needs supply slightly higher than 5v to compare signals close / at 5v.\n\nSpecific voltage was choosen, as it both enabled comparing accross\nthe whole 0-5v band, and resulted in the opamp outputing around 5V as\nlogic-high. (Output of Opamp ist at max aprox. 1.2-1.3 V lower than Supply Voltage)"
Changed lines of the file:
@@
 Vout = aprox 6.2V
 Text Notes 5900 1500 0    50   ~ 0
-OpAmp used as comparator\n needs supply slightly higher than 5v to compare signals close / at 5v.\n\nSpecific voltage was choosen, as it both enabled comparing accross\nthe whole 0-5v band, and resulted in the opamp outputing around 5V as\nlogic-high. (Output of Opamp ist at max aprox. 1.2-1.3 V lower than Supply Voltage)
+OpAmp used as comparator\nneeds supply slightly higher than 5v to compare signals close to / at 5v.\n\nSpecific voltage was choosen as it both enabled comparing accross\nthe whole 0-5v band, and resulted in the opamp outputing around 5V as\nlogic-high. (Output of Opamp ist at max aprox. 1.2-1.3 V lower than Supply Voltage)
 $Comp
 L power:GND #PWR0192

Commit message: Schematic Update First Draft, ERC Passed
Parts:
- added H1, H2: MountingHole, MountingHole:MountingHole_3.2mm_M3_Pad_Via, symbol Mechanical:MountingHole
Changed lines of the file:
@@
 $Descr A4 11693 8268
 encoding utf-8
-Sheet 10 11
+Sheet 6 9
 Title "Schilk_SA-ADC"
 Date "2020-02-03"
@@
 	3050 1350 3050 2900
 Wire Wire Line
-	2450 1350 3050 1350
+	2450 1350 2900 1350
 Connection ~ 3050 1350
 Wire Wire Line
 	2450 1450 2600 1450
-Wire Wire Line
-	2600 1450 2600 1650
 $Comp
 L power:GND #PWR0196
@@
 	1    0    0    -1
 $EndComp
+$Comp
+L Mechanical:MountingHole H1
+U 1 1 606C05C3
+P 4200 4250
+F 0 "H1" H 4300 4296 50  0000 L CNN
+F 1 "MountingHole" H 4300 4205 50  0000 L CNN
+F 2 "MountingHole:MountingHole_3.2mm_M3_Pad_Via" H 4200 4250 50  0001 C CNN
+F 3 "~" H 4200 4250 50  0001 C CNN
+	1    4200 4250
+	1    0    0    -1
+$EndComp
+$Comp
+L Mechanical:MountingHole H2
+U 1 1 606C0E4F
+P 4200 4550
+F 0 "H2" H 4300 4596 50  0000 L CNN
+F 1 "MountingHole" H 4300 4505 50  0000 L CNN
+F 2 "MountingHole:MountingHole_3.2mm_M3_Pad_Via" H 4200 4550 50  0001 C CNN
+F 3 "~" H 4200 4550 50  0001 C CNN
+	1    4200 4550
+	1    0    0    -1
+$EndComp
+$Comp
+L power:PWR_FLAG #FLG0101
+U 1 1 606CF77D
+P 2900 1250
+F 0 "#FLG0101" H 2900 1325 50  0001 C CNN
+F 1 "PWR_FLAG" H 2900 1423 50  0000 C CNN
+F 2 "" H 2900 1250 50  0001 C CNN
+F 3 "~" H 2900 1250 50  0001 C CNN
+	1    2900 1250
+	1    0    0    -1
+$EndComp
+Wire Wire Line
+	2900 1350 2900 1250
+Connection ~ 2900 1350
+Wire Wire Line
+	2900 1350 3050 1350
+$Comp
+L power:PWR_FLAG #FLG0102
+U 1 1 60985617
+P 2500 1600
+F 0 "#FLG0102" H 2500 1675 50  0001 C CNN
+F 1 "PWR_FLAG" V 2500 1727 50  0000 L CNN
+F 2 "" H 2500 1600 50  0001 C CNN
+F 3 "~" H 2500 1600 50  0001 C CNN
+	1    2500 1600
+	0    -1   -1   0
+$EndComp
+Wire Wire Line
+	2500 1600 2600 1600
+Wire Wire Line
+	2600 1450 2600 1600
+Connection ~ 2600 1600
+Wire Wire Line
+	2600 1600 2600 1650
 $EndSCHEMATC

Commit message: PCB v0.2.
Parts:
- J2: value Conn_01x02 -> Power
- U37: value LM317L_TO92 -> LM317
- U38: value L7805 -> L7805CDT
Changed lines of the file:
@@
 P 3550 2900
 F 0 "U38" H 3550 3142 50  0000 C CNN
-F 1 "L7805" H 3550 3051 50  0000 C CNN
+F 1 "L7805CDT" H 3550 3051 50  0000 C CNN
 F 2 "Package_TO_SOT_SMD:TO-252-2" H 3575 2750 50  0001 L CIN
 F 3 "http://www.st.com/content/ccc/resource/technical/document/datasheet/41/4f/b3/b0/12/d4/47/88/CD00000444.pdf/files/CD00000444.pdf/jcr:content/translations/en.CD00000444.pdf" H 3550 2850 50  0001 C CNN
@@
 P 2250 1450
 F 0 "J2" H 2168 1125 50  0000 C CNN
-F 1 "Conn_01x02" H 2168 1216 50  0000 C CNN
+F 1 "Power" H 2168 1216 50  0000 C CNN
 F 2 "Connector_PinHeader_2.54mm:PinHeader_1x02_P2.54mm_Horizontal" H 2250 1450 50  0001 C CNN
 F 3 "~" H 2250 1450 50  0001 C CNN
@@
 P 3550 1350
 F 0 "U37" H 3550 1592 50  0000 C CNN
-F 1 "LM317L_TO92" H 3550 1501 50  0000 C CNN
+F 1 "LM317" H 3550 1501 50  0000 C CNN
 F 2 "Package_TO_SOT_SMD:TO-252-2" H 3550 1575 50  0001 C CIN
 F 3 "http://www.ti.com/lit/ds/snvs775k/snvs775k.pdf" H 3550 1350 50  0001 C CNN
