File: KiCad/StateMaschine.sch (KiCad schematic (older format))
At the start: 28 parts, among them U27 74LVC1G04, U28 74HC164, U29 74LVC1G175, U30 74HC02, U31 74HC02

Commit message: PCB v0.2.
Parts:
- D1, D2, D3, D4, D5, D6, D7, D8, D9: value LED_Small -> LED
- U27: value 74LVC1G04 -> SN74LVC1G04DCK
- U28: value 74HC164 -> 74HC161D
- U29: value 74LVC1G175 -> SN74LVC1G175DCK
- U30: value 74HC02 -> SN74HC02D
- U31: value 74HC02 -> SN74HC08D; symbol 74xx:74HC02 -> 74xx:74LS08
- U31: value 74HC02 -> SN74HC08D
Connections:
- net C_IN: now also U31.8; no longer U31.10
- net GND: now also U31.13; no longer U31.11
- net at U30.1: now also U31.1; no longer U31.2
- net at U30.4: now also U31.2; no longer U31.3
- net at U30.10: now also U31.4; no longer U31.5
- net at U30.13: now also U31.5; no longer U31.6
- net at U31.9: now also U31.3; no longer U31.4
- new net: U31.10, U31.6
Changed lines of the file:
@@
 AR Path="/5E356A03/5E406DA3" Ref="D1"  Part="1"
 F 0 "D1" H 8750 1550 50  0000 C CNN
-F 1 "LED_Small" H 8400 1550 50  0000 C CNN
+F 1 "LED" H 8400 1550 50  0000 C CNN
 F 2 "LED_SMD:LED_0603_1608Metric" V 8650 1600 50  0001 C CNN
 F 3 "~" V 8650 1600 50  0001 C CNN
@@
 AR Path="/5E356A03/5E406DB0" Ref="D2"  Part="1"
 F 0 "D2" H 8750 1650 50  0000 C CNN
-F 1 "LED_Small" H 8400 1650 50  0000 C CNN
+F 1 "LED" H 8400 1650 50  0000 C CNN
 F 2 "LED_SMD:LED_0603_1608Metric" V 8650 1700 50  0001 C CNN
 F 3 "~" V 8650 1700 50  0001 C CNN
@@
 AR Path="/5E356A03/5E406DBD" Ref="D3"  Part="1"
 F 0 "D3" H 8750 1750 50  0000 C CNN
-F 1 "LED_Small" H 8400 1750 50  0000 C CNN
+F 1 "LED" H 8400 1750 50  0000 C CNN
 F 2 "LED_SMD:LED_0603_1608Metric" V 8650 1800 50  0001 C CNN
 F 3 "~" V 8650 1800 50  0001 C CNN
@@
 AR Path="/5E356A03/5E406DCA" Ref="D4"  Part="1"
 F 0 "D4" H 8750 1850 50  0000 C CNN
-F 1 "LED_Small" H 8400 1850 50  0000 C CNN
+F 1 "LED" H 8400 1850 50  0000 C CNN
 F 2 "LED_SMD:LED_0603_1608Metric" V 8650 1900 50  0001 C CNN
 F 3 "~" V 8650 1900 50  0001 C CNN
@@
 AR Path="/5E356A03/5E406DD7" Ref="D5"  Part="1"
 F 0 "D5" H 8750 1950 50  0000 C CNN
-F 1 "LED_Small" H 8400 1950 50  0000 C CNN
+F 1 "LED" H 8400 1950 50  0000 C CNN
 F 2 "LED_SMD:LED_0603_1608Metric" V 8650 2000 50  0001 C CNN
 F 3 "~" V 8650 2000 50  0001 C CNN
@@
 AR Path="/5E356A03/5E406DE4" Ref="D6"  Part="1"
 F 0 "D6" H 8750 2050 50  0000 C CNN
-F 1 "LED_Small" H 8400 2050 50  0000 C CNN
+F 1 "LED" H 8400 2050 50  0000 C CNN
 F 2 "LED_SMD:LED_0603_1608Metric" V 8650 2100 50  0001 C CNN
 F 3 "~" V 8650 2100 50  0001 C CNN
@@
 AR Path="/5E356A03/5E406DF1" Ref="D7"  Part="1"
 F 0 "D7" H 8750 2150 50  0000 C CNN
-F 1 "LED_Small" H 8400 2150 50  0000 C CNN
+F 1 "LED" H 8400 2150 50  0000 C CNN
 F 2 "LED_SMD:LED_0603_1608Metric" V 8650 2200 50  0001 C CNN
 F 3 "~" V 8650 2200 50  0001 C CNN
@@
 AR Path="/5E356A03/5E406DFE" Ref="D8"  Part="1"
 F 0 "D8" H 8750 2250 50  0000 C CNN
-F 1 "LED_Small" H 8400 2250 50  0000 C CNN
+F 1 "LED" H 8400 2250 50  0000 C CNN
 F 2 "LED_SMD:LED_0603_1608Metric" V 8650 2300 50  0001 C CNN
 F 3 "~" V 8650 2300 50  0001 C CNN
@@
 AR Path="/5E356A03/5E411742" Ref="D9"  Part="1"
 F 0 "D9" H 8750 2350 50  0000 C CNN
-F 1 "LED_Small" H 8400 2350 50  0000 C CNN
+F 1 "LED" H 8400 2350 50  0000 C CNN
 F 2 "LED_SMD:LED_0603_1608Metric" V 8650 2400 50  0001 C CNN
 F 3 "~" V 8650 2400 50  0001 C CNN
@@
 P 3750 2000
 F 0 "U28" H 3850 2550 50  0000 C CNN
-F 1 "74HC164" H 3950 2450 50  0000 C CNN
+F 1 "74HC161D" H 4000 2450 50  0000 C CNN
 F 2 "Package_SO:SOIC-14_3.9x8.7mm_P1.27mm" H 4650 1700 50  0001 C CNN
 F 3 "https://assets.nexperia.com/documents/data-sheet/74HC_HCT164.pdf" H 4650 1700 50  0001 C CNN
@@
 P 4600 2950
 F 0 "U29" H 4700 2650 50  0000 C CNN
-F 1 "74LVC1G175" H 4900 2750 50  0000 C CNN
+F 1 "SN74LVC1G175DCK" H 5050 2750 50  0000 C CNN
 F 2 "Package_TO_SOT_SMD:SOT-363_SC-70-6" H 4600 2950 50  0001 C CNN
 F 3 "http://www.ti.com/lit/sg/scyt129e/scyt129e.pdf" H 4600 2950 50  0001 C CNN
@@
 P 2350 2950
 F 0 "U27" H 2500 3150 50  0000 C CNN
-F 1 "74LVC1G04" H 2650 3050 50  0000 C CNN
+F 1 "SN74LVC1G04DCK" H 2650 3050 50  0000 C CNN
 F 2 "Package_TO_SOT_SMD:SOT-353_SC-70-5" H 2350 2950 50  0001 C CNN
 F 3 "http://www.ti.com/lit/sg/scyt129e/scyt129e.pdf" H 2350 2950 50  0001 C CNN
@@
 P 3400 4150
 F 0 "U30" H 3400 4475 50  0000 C CNN
-F 1 "74HC02" H 3400 4384 50  0000 C CNN
+F 1 "SN74HC02D" H 3400 4384 50  0000 C CNN
 F 2 "Package_SO:SOIC-14_3.9x8.7mm_P1.27mm" H 3400 4150 50  0001 C CNN
 F 3 "http://www.ti.com/lit/gpn/sn74hc02" H 3400 4150 50  0001 C CNN
@@
 P 3400 4750
 F 0 "U30" H 3400 5075 50  0000 C CNN
-F 1 "74HC02" H 3400 4984 50  0000 C CNN
+F 1 "SN74HC02D" H 3400 4984 50  0000 C CNN
 F 2 "Package_SO:SOIC-14_3.9x8.7mm_P1.27mm" H 3400 4750 50  0001 C CNN
 F 3 "http://www.ti.com/lit/gpn/sn74hc02" H 3400 4750 50  0001 C CNN
@@
 P 3400 5300
 F 0 "U30" H 3400 5625 50  0000 C CNN
-F 1 "74HC02" H 3400 5534 50  0000 C CNN
+F 1 "SN74HC02D" H 3400 5534 50  0000 C CNN
 F 2 "Package_SO:SOIC-14_3.9x8.7mm_P1.27mm" H 3400 5300 50  0001 C CNN
 F 3 "http://www.ti.com/lit/gpn/sn74hc02" H 3400 5300 50  0001 C CNN
@@
 P 3400 5850
 F 0 "U30" H 3400 6175 50  0000 C CNN
-F 1 "74HC02" H 3400 6084 50  0000 C CNN
+F 1 "SN74HC02D" H 3400 6084 50  0000 C CNN
 F 2 "Package_SO:SOIC-14_3.9x8.7mm_P1.27mm" H 3400 5850 50  0001 C CNN
 F 3 "http://www.ti.com/lit/gpn/sn74hc02" H 3400 5850 50  0001 C CNN
@@
 P 3400 7000
 F 0 "U30" H 3630 7046 50  0000 L CNN
-F 1 "74HC02" H 3630 6955 50  0000 L CNN
+F 1 "SN74HC02D" H 3630 6955 50  0000 L CNN
 F 2 "Package_SO:SOIC-14_3.9x8.7mm_P1.27mm" H 3400 7000 50  0001 C CNN
 F 3 "http://www.ti.com/lit/gpn/sn74hc02" H 3400 7000 50  0001 C CNN
@@
 	2700 4050 3100 4050
 $Comp
-L 74xx:74HC02 U31
+L 74xx:74LS08 U31
 U 1 1 60890547
 P 4650 4100
 F 0 "U31" H 4650 4425 50  0000 C CNN
-F 1 "74HC02" H 4650 4334 50  0000 C CNN
+F 1 "SN74HC08D" H 4650 4334 50  0000 C CNN
 F 2 "Package_SO:SOIC-14_3.9x8.7mm_P1.27mm" H 4650 4100 50  0001 C CNN
 F 3 "http://www.ti.com/lit/gpn/sn74hc02" H 4650 4100 50  0001 C CNN
@@
 $EndComp
 $Comp
-L 74xx:74HC02 U31
+L 74xx:74LS08 U31
 U 2 1 6089054D
 P 4650 4700
 F 0 "U31" H 4650 5025 50  0000 C CNN
-F 1 "74HC02" H 4650 4934 50  0000 C CNN
+F 1 "SN74HC08D" H 4650 4934 50  0000 C CNN
 F 2 "Package_SO:SOIC-14_3.9x8.7mm_P1.27mm" H 4650 4700 50  0001 C CNN
 F 3 "http://www.ti.com/lit/gpn/sn74hc02" H 4650 4700 50  0001 C CNN
@@
 $EndComp
 $Comp
-L 74xx:74HC02 U31
+L 74xx:74LS08 U31
 U 3 1 60890553
 P 4650 5250
 F 0 "U31" H 4900 5150 50  0000 C CNN
-F 1 "74HC02" H 4950 5350 50  0000 C CNN
+F 1 "SN74HC08D" H 5000 5400 50  0000 C CNN
 F 2 "Package_SO:SOIC-14_3.9x8.7mm_P1.27mm" H 4650 5250 50  0001 C CNN
 F 3 "http://www.ti.com/lit/gpn/sn74hc02" H 4650 5250 50  0001 C CNN
@@
 P 4650 7000
 F 0 "U31" H 4880 7046 50  0000 L CNN
-F 1 "74HC02" H 4880 6955 50  0000 L CNN
+F 1 "SN74HC08D" H 4880 6955 50  0000 L CNN
 F 2 "Package_SO:SOIC-14_3.9x8.7mm_P1.27mm" H 4650 7000 50  0001 C CNN
 F 3 "http://www.ti.com/lit/gpn/sn74hc02" H 4650 7000 50  0001 C CNN
@@
 	5150 4100 4950 4100
 $Comp
-L 74xx:74HC02 U31
+L 74xx:74LS08 U31
 U 4 1 60890559
 P 4650 5800
 F 0 "U31" H 4900 5700 50  0000 C CNN
-F 1 "74HC02" H 4950 5950 50  0000 C CNN
+F 1 "SN74HC08D" H 5000 5950 50  0000 C CNN
 F 2 "Package_SO:SOIC-14_3.9x8.7mm_P1.27mm" H 4650 5800 50  0001 C CNN
 F 3 "http://www.ti.com/lit/gpn/sn74hc02" H 4650 5800 50  0001 C CNN

Commit message: v0.3 Changed to Schmitt-Trigger ICs Added pull-down resistor to Clock Enable
Parts:
- R1, R2, R3, R4, R5, R6, R7, R8, R9: value rled -> 39K
Changed lines of the file:
@@
 Sheet 7 9
 Title "Schilk_SA-ADC"
-Date "2020-02-03"
-Rev "v0.0 (Prod.)"
+Date "2020-08-26"
+Rev "v0.3"
 Comp ""
 Comment1 ""
@@
 AR Path="/5E356A03/5E406D9D" Ref="R1"  Part="1"
 F 0 "R1" V 8150 1800 50  0000 C CNN
-F 1 "rled" V 8150 1400 50  0000 C CNN
+F 1 "39K" V 8150 1400 50  0000 C CNN
 F 2 "Resistor_SMD:R_0603_1608Metric" H 8200 1600 50  0001 C CNN
 F 3 "~" H 8200 1600 50  0001 C CNN
@@
 AR Path="/5E356A03/5E406DAA" Ref="R2"  Part="1"
 F 0 "R2" V 8150 1900 50  0000 C CNN
-F 1 "rled" V 8150 1500 50  0000 C CNN
+F 1 "39K" V 8150 1500 50  0000 C CNN
 F 2 "Resistor_SMD:R_0603_1608Metric" H 8200 1700 50  0001 C CNN
 F 3 "~" H 8200 1700 50  0001 C CNN
@@
 AR Path="/5E356A03/5E406DB7" Ref="R3"  Part="1"
 F 0 "R3" V 8150 2000 50  0000 C CNN
-F 1 "rled" V 8150 1600 50  0000 C CNN
+F 1 "39K" V 8150 1600 50  0000 C CNN
 F 2 "Resistor_SMD:R_0603_1608Metric" H 8200 1800 50  0001 C CNN
 F 3 "~" H 8200 1800 50  0001 C CNN
@@
 AR Path="/5E356A03/5E406DC4" Ref="R4"  Part="1"
 F 0 "R4" V 8150 2100 50  0000 C CNN
-F 1 "rled" V 8150 1700 50  0000 C CNN
+F 1 "39K" V 8150 1700 50  0000 C CNN
 F 2 "Resistor_SMD:R_0603_1608Metric" H 8200 1900 50  0001 C CNN
 F 3 "~" H 8200 1900 50  0001 C CNN
@@
 AR Path="/5E356A03/5E406DD1" Ref="R5"  Part="1"
 F 0 "R5" V 8150 2200 50  0000 C CNN
-F 1 "rled" V 8150 1800 50  0000 C CNN
+F 1 "39K" V 8150 1800 50  0000 C CNN
 F 2 "Resistor_SMD:R_0603_1608Metric" H 8200 2000 50  0001 C CNN
 F 3 "~" H 8200 2000 50  0001 C CNN
@@
 AR Path="/5E356A03/5E406DDE" Ref="R6"  Part="1"
 F 0 "R6" V 8150 2300 50  0000 C CNN
-F 1 "rled" V 8150 1900 50  0000 C CNN
+F 1 "39K" V 8150 1900 50  0000 C CNN
 F 2 "Resistor_SMD:R_0603_1608Metric" H 8200 2100 50  0001 C CNN
 F 3 "~" H 8200 2100 50  0001 C CNN
@@
 AR Path="/5E356A03/5E406DEB" Ref="R7"  Part="1"
 F 0 "R7" V 8150 2400 50  0000 C CNN
-F 1 "rled" V 8150 2000 50  0000 C CNN
+F 1 "39K" V 8150 2000 50  0000 C CNN
 F 2 "Resistor_SMD:R_0603_1608Metric" H 8200 2200 50  0001 C CNN
 F 3 "~" H 8200 2200 50  0001 C CNN
@@
 AR Path="/5E356A03/5E406DF8" Ref="R8"  Part="1"
 F 0 "R8" V 8150 2500 50  0000 C CNN
-F 1 "rled" V 8150 2100 50  0000 C CNN
+F 1 "39K" V 8150 2100 50  0000 C CNN
 F 2 "Resistor_SMD:R_0603_1608Metric" H 8200 2300 50  0001 C CNN
 F 3 "~" H 8200 2300 50  0001 C CNN
@@
 AR Path="/5E356A03/5E41173C" Ref="R9"  Part="1"
 F 0 "R9" V 8150 2600 50  0000 C CNN
-F 1 "rled" V 8150 2200 50  0000 C CNN
+F 1 "39K" V 8150 2200 50  0000 C CNN
 F 2 "Resistor_SMD:R_0603_1608Metric" H 8200 2400 50  0001 C CNN
 F 3 "~" H 8200 2400 50  0001 C CNN
